File: Flight_Controller/Flight_Controller.kicad_pcb (KiCad board)
At the start: 2 copper layers, 123 parts, among them IC1 ICM-20689, J1 USB_C_Receptacle_USB2.0_16P, J2 SM08B-SRSS-TB, J3 SM04B-SRSS-TB, J4 SM06B-SRSS-TBLFSN, J5 SM03B-SRSS-TB, Q1 AO3400A, SW1 SW_Push, U1 NO, U11 ESD224DQA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

Commit message: Primer emplazamiento
Parts:
- C9, D1, U5: moved to B.Cu
- moved J2 185.7 mm to (212.2, 84.0), turned to 90 degrees
- moved U2 171.4 mm to (195.0, 89.5), turned to -90 degrees
- moved U3 164.3 mm to (189.5, 76.0), turned to -90 degrees
- moved R1 161.7 mm to (194.0, 83.0), turned to -90 degrees
- moved C6 160.6 mm to (184.5, 101.5), turned to 90 degrees
- moved R3 159.3 mm to (195.0, 75.5), turned to -90 degrees
- moved J1 159.1 mm to (192.0, 68.5), turned to 180 degrees
- moved R4 159.0 mm to (193.5, 75.5), turned to -90 degrees
- moved R8 158.1 mm to (173.8, 79.0)
- moved R2 157.9 mm to (195.5, 95.5), turned to 90 degrees
- moved C4 157.6 mm to (183.0, 103.5), turned to -90 degrees
- moved U49 155.2 mm to (167.5, 81.0), turned to 180 degrees
- moved C3 154.5 mm to (181.0, 104.5), turned to 180 degrees
- moved C2 154.3 mm to (181.0, 103.0), turned to 180 degrees
- moved R22 151.1 mm to (190.5, 79.0), turned to -90 degrees
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